File: attiny85-sensor.kicad_pcb (KiCad board)
At the start: 2 copper layers, 27.9 x 30.5 mm, 11 parts, among them IC1 ATTINY85-P, P1 PIR, P2 BIND_BTN, P3 CONN_01X02, P4 CONN_01X06

Commit message: Socket for the chip
Parts:
- IC1: footprint Housings_DIP:DIP-8_W7.62mm -> Housings_DIP:DIP-8_W7.62mm_Socket
Changed lines of the file:
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@@
-(kicad_pcb (version 4) (host pcbnew 4.0.5+dfsg1-4)
+(kicad_pcb (version 4) (host pcbnew 4.0.7-e2-6376~58~ubuntu16.04.1)
   (general
     (links 26)
     (no_connects 0)
-    (area 155.84 88.646666 188.625 122.67)
+    (area 158.674999 90.094999 186.765001 120.725001)
     (thickness 1.6)
     (drawings 10)
@@
     (add_net Earth)
   )
-  (module Housings_DIP:DIP-8_W7.62mm (layer F.Cu)
-    (at 168.91 105.41)
-    (descr "8-lead dip package, row spacing 7.62 mm (300 mils)")
-    (tags "dil dip 2.54 300")
-    (fp_text reference IC1 (at 3.81 8.89) (layer F.SilkS)
-      (effects (font (size 1 1) (thickness 0.15)))
-    )
-    (fp_text value ATTINY85-P (at 0 -3.72) (layer F.Fab)
-      (effects (font (size 1 1) (thickness 0.15)))
-    )
-    (fp_line (start -1.05 -2.45) (end -1.05 10.1) (layer F.CrtYd) (width 0.05))
-    (fp_line (start 8.65 -2.45) (end 8.65 10.1) (layer F.CrtYd) (width 0.05))
-    (fp_line (start -1.05 -2.45) (end 8.65 -2.45) (layer F.CrtYd) (width 0.05))
-    (fp_line (start -1.05 10.1) (end 8.65 10.1) (layer F.CrtYd) (width 0.05))
-    (fp_line (start 0.135 -2.295) (end 0.135 -1.025) (layer F.SilkS) (width 0.15))
-    (fp_line (start 7.485 -2.295) (end 7.485 -1.025) (layer F.SilkS) (width 0.15))
-    (fp_line (start 7.485 9.915) (end 7.485 8.645) (layer F.SilkS) (width 0.15))
-    (fp_line (start 0.135 9.915) (end 0.135 8.645) (layer F.SilkS) (width 0.15))
-    (fp_line (start 0.135 -2.295) (end 7.485 -2.295) (layer F.SilkS) (width 0.15))
-    (fp_line (start 0.135 9.915) (end 7.485 9.915) (layer F.SilkS) (width 0.15))
-    (fp_line (start 0.135 -1.025) (end -0.8 -1.025) (layer F.SilkS) (width 0.15))
-    (pad 1 thru_hole oval (at 0 0) (size 1.6 1.6) (drill 0.8) (layers *.Cu *.Mask)
-      (net 6 "Net-(IC1-Pad1)"))
-    (pad 2 thru_hole oval (at 0 2.54) (size 1.6 1.6) (drill 0.8) (layers *.Cu *.Mask)
-      (net 3 "Net-(IC1-Pad2)"))
-    (pad 3 thru_hole oval (at 0 5.08) (size 1.6 1.6) (drill 0.8) (layers *.Cu *.Mask)
-      (net 4 "Net-(IC1-Pad3)"))
-    (pad 4 thru_hole oval (at 0 7.62) (size 1.6 1.6) (drill 0.8) (layers *.Cu *.Mask)
-      (net 2 Earth))
-    (pad 5 thru_hole oval (at 7.62 7.62) (size 1.6 1.6) (drill 0.8) (layers *.Cu *.Mask)
-      (net 7 "Net-(IC1-Pad5)"))
-    (pad 6 thru_hole oval (at 7.62 5.08) (size 1.6 1.6) (drill 0.8) (layers *.Cu *.Mask)
-      (net 10 "Net-(D1-Pad2)"))
-    (pad 7 thru_hole oval (at 7.62 2.54) (size 1.6 1.6) (drill 0.8) (layers *.Cu *.Mask)
-      (net 8 "Net-(IC1-Pad7)"))
-    (pad 8 thru_hole oval (at 7.62 0) (size 1.6 1.6) (drill 0.8) (layers *.Cu *.Mask)
-      (net 1 +3V3))
-    (model Housings_DIP.3dshapes/DIP-8_W7.62mm.wrl
-      (at (xyz 0 0 0))
-      (scale (xyz 1 1 1))
-      (rotate (xyz 0 0 0))
-    )
-  )
   (module Discret:C1V8 (layer F.Cu)
     (at 172.72 93.98 180)
@@
       (at (xyz 0 0 0))
       (scale (xyz 1 1 1))
+      (rotate (xyz 0 0 0))
+    )
+  )
+  (module Housings_DIP:DIP-8_W7.62mm_Socket (layer F.Cu)
+    (at 168.91 105.41)
+    (descr "8-lead though-hole mounted DIP package, row spacing 7.62 mm (300 mils), Socket")
+    (tags "THT DIP DIL PDIP 2.54mm 7.62mm 300mil Socket")
+    (fp_text reference IC1 (at 3.81 -2.33) (layer F.SilkS)
+      (effects (font (size 1 1) (thickness 0.15)))
+    )
+    (fp_text value ATTINY85-P (at 3.81 9.95) (layer F.Fab)
+      (effects (font (size 1 1) (thickness 0.15)))
+    )
+    (fp_arc (start 3.81 -1.33) (end 2.81 -1.33) (angle -180) (layer F.SilkS) (width 0.12))
+    (fp_line (start 1.635 -1.27) (end 6.985 -1.27) (layer F.Fab) (width 0.1))
+    (fp_line (start 6.985 -1.27) (end 6.985 8.89) (layer F.Fab) (width 0.1))
+    (fp_line (start 6.985 8.89) (end 0.635 8.89) (layer F.Fab) (width 0.1))
+    (fp_line (start 0.635 8.89) (end 0.635 -0.27) (layer F.Fab) (width 0.1))
+    (fp_line (start 0.635 -0.27) (end 1.635 -1.27) (layer F.Fab) (width 0.1))
+    (fp_line (start -1.27 -1.33) (end -1.27 8.95) (layer F.Fab) (width 0.1))
+    (fp_line (start -1.27 8.95) (end 8.89 8.95) (layer F.Fab) (width 0.1))
+    (fp_line (start 8.89 8.95) (end 8.89 -1.33) (layer F.Fab) (width 0.1))
+    (fp_line (start 8.89 -1.33) (end -1.27 -1.33) (layer F.Fab) (width 0.1))
+    (fp_line (start 2.81 -1.33) (end 1.16 -1.33) (layer F.SilkS) (width 0.12))
+    (fp_line (start 1.16 -1.33) (end 1.16 8.95) (layer F.SilkS) (width 0.12))
+    (fp_line (start 1.16 8.95) (end 6.46 8.95) (layer F.SilkS) (width 0.12))
+    (fp_line (start 6.46 8.95) (end 6.46 -1.33) (layer F.SilkS) (width 0.12))
+    (fp_line (start 6.46 -1.33) (end 4.81 -1.33) (layer F.SilkS) (width 0.12))
+    (fp_line (start -1.33 -1.39) (end -1.33 9.01) (layer F.SilkS) (width 0.12))
+    (fp_line (start -1.33 9.01) (end 8.95 9.01) (layer F.SilkS) (width 0.12))
+    (fp_line (start 8.95 9.01) (end 8.95 -1.39) (layer F.SilkS) (width 0.12))
+    (fp_line (start 8.95 -1.39) (end -1.33 -1.39) (layer F.SilkS) (width 0.12))
+    (fp_line (start -1.55 -1.6) (end -1.55 9.2) (layer F.CrtYd) (width 0.05))
+    (fp_line (start -1.55 9.2) (end 9.15 9.2) (layer F.CrtYd) (width 0.05))
+    (fp_line (start 9.15 9.2) (end 9.15 -1.6) (layer F.CrtYd) (width 0.05))
+    (fp_line (start 9.15 -1.6) (end -1.55 -1.6) (layer F.CrtYd) (width 0.05))
+    (fp_text user %R (at 3.81 3.81) (layer F.Fab)
+      (effects (font (size 1 1) (thickness 0.15)))
+    )
+    (pad 1 thru_hole rect (at 0 0) (size 1.6 1.6) (drill 0.8) (layers *.Cu *.Mask)
+      (net 6 "Net-(IC1-Pad1)"))
+    (pad 5 thru_hole oval (at 7.62 7.62) (size 1.6 1.6) (drill 0.8) (layers *.Cu *.Mask)
+      (net 7 "Net-(IC1-Pad5)"))
+    (pad 2 thru_hole oval (at 0 2.54) (size 1.6 1.6) (drill 0.8) (layers *.Cu *.Mask)
+      (net 3 "Net-(IC1-Pad2)"))
+    (pad 6 thru_hole oval (at 7.62 5.08) (size 1.6 1.6) (drill 0.8) (layers *.Cu *.Mask)
+      (net 10 "Net-(D1-Pad2)"))
+    (pad 3 thru_hole oval (at 0 5.08) (size 1.6 1.6) (drill 0.8) (layers *.Cu *.Mask)
+      (net 4 "Net-(IC1-Pad3)"))
+    (pad 7 thru_hole oval (at 7.62 2.54) (size 1.6 1.6) (drill 0.8) (layers *.Cu *.Mask)
+      (net 8 "Net-(IC1-Pad7)"))
+    (pad 4 thru_hole oval (at 0 7.62) (size 1.6 1.6) (drill 0.8) (layers *.Cu *.Mask)
+      (net 2 Earth))
+    (pad 8 thru_hole oval (at 7.62 0) (size 1.6 1.6) (drill 0.8) (layers *.Cu *.Mask)
+      (net 1 +3V3))
+    (model ${KISYS3DMOD}/Housings_DIP.3dshapes/DIP-8_W7.62mm_Socket.wrl
+      (at (xyz 0 0 0))
+      (scale (xyz 1 1 1))
